Commit message: fix mass value for helios 16p

File: urdf/rs_helios_16p.urdf.xacro (robot description, xacro)
@@ -25,5 +25,5 @@
       <xacro:if value="${include_inertial}">
         <inertial>
-          <mass value="100.840" />
+          <mass value="1.0" />
           <origin xyz="0 0 0.04135" />
 			  	<xacro:solid_cuboid_inertia m="0.840" w="0.109" h="0.109" d="0.0827" />
