Commit message: Normalize axis, camera topics, zoom for link750

File: urdf/link_750_nh.urdf.xacro (robot description, xacro)
@@ -7,7 +7,7 @@
   <xacro:property name="ptz_mechanical_reduction" value="1.0"/>
   <xacro:property name="PI" value="3.14159265359"/>
-  <xacro:macro name="sensor_link_750_nh" params="prefix parent *origin far:=^|8.0 near:=^|0.05 prefix_topic:=^ptz_camera include_inertial:=^|true">
+  <xacro:macro name="sensor_link_750_nh" params="prefix parent *origin far:=^|8.0 near:=^|0.05 prefix_topic:=^ptz_camera include_inertial:=^|true fps:=^|30.0">
     <joint name="${prefix}_joint" type="fixed">
-      <axis xyz="0 1 0"/>
+      <axis xyz="0 0 1"/>
       <xacro:insert_block name="origin"/>
       <parent link="${parent}"/>
@@ -39,5 +39,5 @@
     </link>
     <joint name="${prefix}_pan_joint" type="revolute">
-      <axis xyz="0 0 -1"/>
+      <axis xyz="0 0 1"/>
       <origin xyz="0.0 0.0 0.0318" rpy="0 0 0"/>
       <!-- check the displacement -->
@@ -82,6 +82,6 @@
     </transmission>
     <joint name="${prefix}_tilt_joint" type="revolute">
-      <axis xyz="0 -1 0"/>
-      <origin xyz="0.0 0.0 0.102" rpy="0 0 0"/>
+      <axis xyz="0 0 1"/>
+      <origin xyz="0.0 0.0 0.102" rpy="${PI/2} 0 0"/>
       <parent link="${prefix}_pan_link"/>
       <child link="${prefix}_tilt_link"/>
@@ -98,5 +98,5 @@
       </xacro:if>
       <visual>
-        <origin xyz="0 0 0" rpy="0 0 0"/>
+        <origin xyz="0 0 0" rpy="${PI/2} 0 0"/>
         <material name="grey_color">
           <color rgba="0.1 0.1 0.1 1"/>
@@ -107,5 +107,5 @@
       </visual>
       <collision>
-        <origin xyz="0.0 0.0 0" rpy="0 0 0"/>
+        <origin xyz="0.0 0.0 0" rpy="${PI/2} 0 0"/>
         <geometry>
           <mesh filename="package://robotnik_sensors/meshes/link_750_tilt.stl" scale="1.0 1.0 1.0"/>
@@ -123,6 +123,32 @@
       </actuator>
     </transmission>
+    <joint name="${prefix}_zoom_joint" type="prismatic">
+      <axis xyz="0 0 1"/>
+      <origin xyz="0.0 0.0 0.0" rpy="0 0 0"/>
+      <parent link="${prefix}_optical_frame_link"/>
+      <child link="${prefix}_zoom_link"/>
+      <limit effort="1000.0" velocity="1" lower="0" upper="10000"/>
+    </joint>
+    <link name="${prefix}_zoom_link">
+      <xacro:if value="${include_inertial}">
+        <inertial>
+          <mass value="0.1"/>
+          <origin xyz="0 0 0" rpy="0 0 0"/>
+          <xacro:solid_cuboid_inertia m="0.1" w="0.11" h="0.11" d="0.1" />
+        </inertial>
+      </xacro:if>
+    </link>
+    <transmission name="${prefix}_zoom_trans">
+      <type>transmission_interface/SimpleTransmission</type>
+      <joint name="${prefix}_zoom_joint">
+        <hardwareInterface>hardware_interface/PositionJointInterface</hardwareInterface>
+      </joint>
+      <actuator name="${prefix}zoom_motor">
+        <hardwareInterface>hardware_interface/PositionJointInterface</hardwareInterface>
+        <mechanicalReduction>1</mechanicalReduction>
+      </actuator>
+    </transmission>
     <joint name="${prefix}_frame_joint" type="fixed">
-      <origin xyz="0 0 0" rpy="0 0 0"/>
+      <origin xyz="0.06 0 0" rpy="${-PI/2} 0 0"/>
       <parent link="${prefix}_tilt_link"/>
       <child link="${prefix}_frame_link"/>
@@ -137,7 +163,7 @@
       </xacro:if>
     </link>
-    <!-- Optical frame -->
+    <!-- Optical frame ${-M_PI/2} -->
     <joint name="${prefix}_optical_joint" type="fixed">
-      <origin xyz="0.02 0 0" rpy="0 0 0"/>
+      <origin xyz="0.0 0 0" rpy="${-M_PI/2} 0 ${-M_PI/2}"/>
       <parent link="${prefix}_frame_link"/>
       <child link="${prefix}_optical_frame_link"/>
@@ -159,7 +185,7 @@
   </xacro:macro>
   <xacro:macro name="sensor_link_750_nh_gazebo">
-    <gazebo reference="${prefix}_optical_frame_link"> <!-- the image will be generated from this (${name}_frame) point of view, with the front being the X axis -->
+    <gazebo reference="${prefix}_frame_link"> <!-- the image will be generated from this (${name}_frame) point of view, with the front being the X axis -->
       <sensor type="camera" name="${prefix}_sensor">
-        <update_rate>30.0</update_rate>
+        <update_rate>${fps}</update_rate>
         <camera name="${prefix_topic}">
           <horizontal_fov>${60.0*M_PI/180.0}</horizontal_fov>
@@ -177,5 +203,5 @@
           <alwaysOn>true</alwaysOn>
           <updateRate>0.0</updateRate>
-          <cameraName>top_rgb_${prefix_topic}</cameraName>
+          <cameraName>${prefix_topic}/rgb</cameraName>
           <imageTopicName>image_raw</imageTopicName>
           <cameraInfoTopicName>camera_info</cameraInfoTopicName>
@@ -193,5 +219,5 @@
       </sensor>
       <sensor type="camera" name="thermal_${prefix}_sensor">
-        <update_rate>30.0</update_rate>
+        <update_rate>${fps}</update_rate>
         <camera>
           <horizontal_fov>${60.0*M_PI/180.0}</horizontal_fov>
@@ -208,9 +234,9 @@
         <plugin name="thermal_camera_controller" filename="libgazebo_ros_thermal_camera.so">
           <alwaysOn>true</alwaysOn>
-          <updateRate>10</updateRate>
-          <cameraName>top_thermal_${prefix_topic}</cameraName>
+          <updateRate>${fps}</updateRate>
+          <cameraName>${prefix_topic}/thermal</cameraName>
           <imageTopicName>image_raw</imageTopicName>
           <cameraInfoTopicName>camera_info</cameraInfoTopicName>
-          <frameName>${prefix}_optical_frame_link</frameName>
+          <frameName>${prefix}_frame_link</frameName>
         </plugin>
       </sensor>
