Commit message: Normalize optical frame & add fps arg for m5525

File: urdf/axis_m5525.urdf.xacro (robot description, xacro)
@@ -7,5 +7,5 @@
   <xacro:property name="ptz_mechanical_reduction" value="1.0"/>
   <xacro:property name="PI" value="3.14159265359"/>
-  <xacro:macro name="sensor_axis_m5525" params="prefix parent *origin far:=^|8.0 near:=^|0.05 prefix_topic:=^ptz_camera include_inertial:=^|true">
+  <xacro:macro name="sensor_axis_m5525" params="prefix parent *origin far:=^|8.0 near:=^|0.05 prefix_topic:=^ptz_camera include_inertial:=^|true fps:=^|30.0">
     <joint name="${prefix}_joint" type="fixed">
       <axis xyz="0 0 1"/>
@@ -41,5 +41,5 @@
     <joint name="${prefix}_pan_joint" type="revolute">
       <axis xyz="0 0 1"/>
-      <origin xyz="0 0.0 0.087" rpy="0 0 0"/>
+      <origin xyz="0 0.0 0.067" rpy="0 0 0"/>
       <!-- check the displacement -->
       <parent link="${prefix}_base_link"/>
@@ -72,5 +72,5 @@
       <parent link="${prefix}_pan_link"/>
       <child link="${prefix}_tilt_link"/>
-      <limit effort="${ptz_joint_effort_limit}" velocity="${ptz_joint_velocity_limit}" lower="-1.5708" upper="1.5708"/>
+      <limit effort="${ptz_joint_effort_limit}" velocity="${ptz_joint_velocity_limit}" lower="0" upper="1.5708"/>
       <joint_properties damping="${ptz_joint_damping}" friction="{ptz_joint_friction}"/>
     </joint>
@@ -95,10 +95,9 @@
     </transmission>
     <joint name="${prefix}_zoom_joint" type="prismatic">
-      <axis xyz="1 0 0"/>
-      <origin xyz="0.0 0.0 0.0" rpy="${-PI/2} 0 0"/>
-      <parent link="${prefix}_tilt_link"/>
+      <axis xyz="0 0 1"/>
+      <origin xyz="0.0 0.0 0.0" rpy="0 0 0"/>
+      <parent link="${prefix}_optical_frame_link"/>
       <child link="${prefix}_zoom_link"/>
-      <limit effort="${ptz_joint_effort_limit}" velocity="${ptz_joint_velocity_limit}" lower="-1.5708" upper="1.5708"/>
-      <joint_properties damping="${ptz_joint_damping}" friction="{ptz_joint_friction}"/>
+      <limit effort="1000.0" velocity="1" lower="0" upper="10000"/>
     </joint>
     <link name="${prefix}_zoom_link">
@@ -118,9 +117,9 @@
       <actuator name="${prefix}zoom_motor">
         <hardwareInterface>hardware_interface/PositionJointInterface</hardwareInterface>
-        <mechanicalReduction>${ptz_mechanical_reduction}</mechanicalReduction>
+        <mechanicalReduction>1</mechanicalReduction>
       </actuator>
     </transmission>
     <joint name="${prefix}_frame_joint" type="fixed">
-      <origin xyz="0 0 0" rpy="0 0 0"/>
+      <origin xyz="0.03 0 0" rpy="${-PI/2} 0 0"/>
       <parent link="${prefix}_tilt_link"/>
       <child link="${prefix}_frame_link"/>
@@ -159,5 +158,5 @@
 		<gazebo reference="${prefix}_frame_link"> <!-- the image will be generated from this (${name}_frame) point of view, with the front being the X axis -->
 			<sensor type="camera" name="${prefix}_sensor">
-				<update_rate>30.0</update_rate>
+				<update_rate>${fps}</update_rate>
 				<camera name="${prefix_topic}">
 					<horizontal_fov>${60.0*M_PI/180.0}</horizontal_fov>

Commit message: Fix ptz zoom joint inertias

File: urdf/axis_m5525.urdf.xacro (robot description, xacro)
@@ -1,5 +1,5 @@
 <?xml version="1.0"?>
 <robot xmlns:xacro="http://wiki.ros.org/xacro" name="sensor_axis_m5525">
-  <xacro:property name="ptz_joint_effort_limit" value="1.0"/>
+  <xacro:property name="ptz_joint_effort_limit" value="10000.0"/>
   <xacro:property name="ptz_joint_velocity_limit" value="1.0"/>
   <xacro:property name="ptz_joint_friction" value="0.1"/>
@@ -99,12 +99,12 @@
       <parent link="${prefix}_optical_frame_link"/>
       <child link="${prefix}_zoom_link"/>
-      <limit effort="1000.0" velocity="1" lower="0" upper="10000"/>
+      <limit effort="10000.0" velocity="5" lower="0" upper="10000"/>
     </joint>
     <link name="${prefix}_zoom_link">
       <xacro:if value="${include_inertial}">
         <inertial>
-          <mass value="0.1"/>
+          <mass value="0.00001"/>
           <origin xyz="0 0 0" rpy="0 0 0"/>
-          <xacro:solid_cuboid_inertia m="0.1" w="0.11" h="0.11" d="0.1" />
+          <xacro:solid_cuboid_inertia m="0.00001" w="0.11" h="0.11" d="0.1" />
         </inertial>
       </xacro:if>

File: urdf/axis_p5676.urdf.xacro (robot description, xacro)
@@ -1,5 +1,5 @@
 <?xml version="1.0"?>
 <robot xmlns:xacro="http://wiki.ros.org/xacro" name="sensor_axis_p5676">
-  <xacro:property name="ptz_joint_effort_limit" value="1.0"/>
+  <xacro:property name="ptz_joint_effort_limit" value="10000.0"/>
   <xacro:property name="ptz_joint_velocity_limit" value="1.0"/>
   <xacro:property name="ptz_joint_friction" value="0.1"/>
@@ -99,12 +99,12 @@
       <parent link="${prefix}_optical_frame_link"/>
       <child link="${prefix}_zoom_link"/>
-      <limit effort="1000.0" velocity="1" lower="0" upper="10000"/>
+      <limit effort="10000.0" velocity="5" lower="0" upper="10000"/>
     </joint>
     <link name="${prefix}_zoom_link">
       <xacro:if value="${include_inertial}">
         <inertial>
-          <mass value="0.1"/>
+          <mass value="0.00001"/>
           <origin xyz="0 0 0" rpy="0 0 0"/>
-          <xacro:solid_cuboid_inertia m="0.1" w="0.11" h="0.11" d="0.1" />
+          <xacro:solid_cuboid_inertia m="0.00001" w="0.11" h="0.11" d="0.1" />
         </inertial>
       </xacro:if>

File: urdf/link_750_nh.urdf.xacro (robot description, xacro)
@@ -1,5 +1,5 @@
 <?xml version="1.0"?>
 <robot xmlns:xacro="http://wiki.ros.org/xacro" name="sensor_link_750_nh">
-  <xacro:property name="ptz_joint_effort_limit" value="1.0"/>
+  <xacro:property name="ptz_joint_effort_limit" value="10000.0"/>
   <xacro:property name="ptz_joint_velocity_limit" value="1.0"/>
   <xacro:property name="ptz_joint_friction" value="0.1"/>
@@ -128,12 +128,12 @@
       <parent link="${prefix}_optical_frame_link"/>
       <child link="${prefix}_zoom_link"/>
-      <limit effort="1000.0" velocity="1" lower="0" upper="10000"/>
+      <limit effort="10000.0" velocity="5" lower="0" upper="10000"/>
     </joint>
     <link name="${prefix}_zoom_link">
       <xacro:if value="${include_inertial}">
         <inertial>
-          <mass value="0.1"/>
+          <mass value="0.00001"/>
           <origin xyz="0 0 0" rpy="0 0 0"/>
-          <xacro:solid_cuboid_inertia m="0.1" w="0.11" h="0.11" d="0.1" />
+          <xacro:solid_cuboid_inertia m="0.00001" w="0.11" h="0.11" d="0.1" />
         </inertial>
       </xacro:if>
