Commit message: Update several plugins for ignition

File: robotnik_sensors/urdf/2d_lidar/sick_nanoscan3.urdf.xacro (robot description, xacro)
@@ -52,9 +52,10 @@
       </xacro:unless>
       <gazebo reference="${frame_prefix}link">
-        <sensor type="${ray_type}" name="${frame_prefix}sensor">
+        <sensor type="gpu_lidar" name="${frame_prefix}sensor">
+          <topic>scan</topic>
           <pose>0.0 0.0 0.0 0.0 0.0 0.0</pose>
           <visualize>false</visualize>
 		  <update_rate>12.5</update_rate>
-          <ray>
+          <lidar>
             <scan>
               <horizontal>
@@ -75,13 +76,5 @@
               <stddev>0.01</stddev>
             </noise>
-          </ray>
-          <plugin name="${node_name}" filename="libgazebo_ros_ray_sensor.so">
-            <ros>
-              <namespace>${node_namespace}</namespace>
-              <remapping>~/out:=~/scan</remapping>
-            </ros>
-            <output_type>sensor_msgs/LaserScan</output_type>
-            <frame_name>${node_namespace}/${frame_prefix}link</frame_name>
-          </plugin>
+          </lidar>
         </sensor>
       </gazebo>

File: robotnik_sensors/urdf/imu/vectornav.urdf.xacro (robot description, xacro)
@@ -114,12 +114,5 @@
           </linear_acceleration>
         </imu>
-        <plugin name="${node_name}" filename="libgazebo_ros_imu_sensor.so">
-          <ros>
-            <namespace>${node_namespace}</namespace>
-            <remapping>~/out:=${topic_prefix}data</remapping>
-          </ros>
-          <initial_orientation_as_reference>false</initial_orientation_as_reference>
-          <frame_name>${node_namespace}/${frame_prefix}link</frame_name>
-        </plugin>
+        <topic>imu</topic>
       </sensor>
     </gazebo>

File: robotnik_sensors/urdf/intel_d435.urdf.xacro (robot description, xacro)
@@ -45,5 +45,5 @@
         <geometry>
           <!-- <box size="${d435_cam_width} ${d435_cam_height} ${d435_cam_depth}"/> -->
-          <mesh filename="package://robotnik_sensors/meshes/intel_d435_color.dae" />
+          <mesh filename="package://robotnik_sensors/meshes/depth/intel_realsense_d435/intel_d435_color.dae" />
         </geometry>
       </visual>
@@ -141,4 +141,5 @@
      <min_depth>0</min_depth>-->
      <sensor name="${camera_name}color" type="camera">
+       <topic>camera/image_raw</topic>
        <camera name="${camera_name}">
          <horizontal_fov>${69.4*deg_to_rad}</horizontal_fov>
@@ -207,4 +208,5 @@
      </sensor>
      <sensor name="${camera_name}depth" type="depth">
+       <topic>camera/depth_image</topic>
        <camera name="${camera_name}">
          <horizontal_fov>${85.2*deg_to_rad}</horizontal_fov>
@@ -227,29 +229,4 @@
        <visualize>false</visualize>
      </sensor>
-   </gazebo>
-   <gazebo>
-     <plugin name="${topics_ns}" filename="librealsense_gazebo_plugin.so">
-       <prefix>${camera_name}</prefix>
-       <depthUpdateRate>60.0</depthUpdateRate>
-       <colorUpdateRate>60.0</colorUpdateRate>
-       <infraredUpdateRate>60.0</infraredUpdateRate>
-       <depthTopicName>${prefix_topic}/depth/image_raw</depthTopicName>
-       <depthCameraInfoTopicName>${prefix_topic}/depth/camera_info</depthCameraInfoTopicName>
-       <colorTopicName>${prefix_topic}/color/image_raw</colorTopicName>
-       <colorCameraInfoTopicName>${prefix_topic}/color/camera_info</colorCameraInfoTopicName>
-       <infrared1TopicName>${prefix_topic}/infra1/image_rect_raw</infrared1TopicName>
-       <infrared1CameraInfoTopicName>${prefix_topic}/infra1/camera_info</infrared1CameraInfoTopicName>
-       <infrared2TopicName>${prefix_topic}/infra2/image_rect_raw</infrared2TopicName>
-       <infrared2CameraInfoTopicName>${prefix_topic}/infra2/camera_info</infrared2CameraInfoTopicName>
-       <colorOpticalframeName>${color_optical_frame}</colorOpticalframeName>
-       <depthOpticalframeName>${depth_optical_frame}</depthOpticalframeName>
-       <infrared1OpticalframeName>${infrared1_optical_frame}</infrared1OpticalframeName>
-       <infrared2OpticalframeName>${infrared2_optical_frame}</infrared2OpticalframeName>
-       <rangeMinDepth>0.2</rangeMinDepth>
-       <rangeMaxDepth>10.0</rangeMaxDepth>
-       <pointCloud>false</pointCloud>
-       <pointCloudTopicName>${prefix_topic}/depth/color/points</pointCloudTopicName>
-       <pointCloudCutoff>0.5</pointCloudCutoff>
-     </plugin>
    </gazebo>
   </xacro:macro>

Commit message: Update sensors configuration for fortress

File: robotnik_sensors/urdf/2d_lidar/sick_nanoscan3.urdf.xacro (robot description, xacro)
@@ -2,5 +2,5 @@
 <robot name="sensor_sick_nanoscan3" xmlns:xacro="http://wiki.ros.org/xacro">
   <xacro:macro name="sensor_sick_nanoscan3"
-               params="frame_prefix
+    params="frame_prefix
                        parent
                        *origin
@@ -12,22 +12,22 @@
     <!-- node_namespace is used from node_name if not set -->
     <xacro:if value="${node_namespace == None}">
-      <xacro:property name="node_namespace" value="${node_name}"/>
+      <xacro:property name="node_namespace" value="${node_name}" />
     </xacro:if>
     <joint name="${frame_prefix}base_joint" type="fixed">
       <xacro:insert_block name="origin" />
-      <parent link="${parent}"/>
-      <child link="${frame_prefix}base_link"/>
+      <parent link="${parent}" />
+      <child link="${frame_prefix}base_link" />
     </joint>
     <link name="${frame_prefix}base_link">
       <visual>
-        <origin xyz="0 0 0" rpy="0 0 0"/>
+        <origin xyz="0 0 0" rpy="0 0 0" />
         <geometry>
-		  <mesh filename="package://robotnik_sensors/meshes/2d_lidar/sick/nanoscan3.stl"/>
+          <mesh filename="package://robotnik_sensors/meshes/2d_lidar/sick/nanoscan3.stl" />
         </geometry>
       </visual>
       <collision>
-        <origin xyz="0 0 0" rpy="0 0 0"/>
+        <origin xyz="0 0 0" rpy="0 0 0" />
         <geometry>
-		  <mesh filename="package://robotnik_sensors/meshes/2d_lidar/sick/nanoscan3.stl"/>
+          <mesh filename="package://robotnik_sensors/meshes/2d_lidar/sick/nanoscan3.stl" />
         </geometry>
       </collision>
@@ -36,26 +36,28 @@
         <origin xyz="0 0 0.04" rpy="0 0 0" />
         <xacro:solid_cuboid_inertia m="0.67" w="0.1006" h="0.1006" d="0.08" />
-	  </inertial>
+      </inertial>
     </link>
     <joint name="${frame_prefix}joint" type="fixed">
-      <origin xyz="0.0 0 0.0505" rpy="0 0 0"/>
-      <parent link="${frame_prefix}base_link"/>
-      <child link="${frame_prefix}link"/>
+      <origin xyz="0.0 0 0.0505" rpy="0 0 0" />
+      <parent link="${frame_prefix}base_link" />
+      <child link="${frame_prefix}link" />
     </joint>
-    <link name="${frame_prefix}link"/>
+    <link name="${frame_prefix}link" />
     <xacro:if value="${simulation}">
-      <xacro:if value="${gpu}">
-        <xacro:property name="ray_type" value="gpu_ray" />
-      </xacro:if>
-      <xacro:unless value="${gpu}">
-        <xacro:property name="ray_type" value="ray" />
-      </xacro:unless>
+      <!-- <xacro:if value="${gpu}"> -->
+      <!--   <xacro:property name="ray_type" value="gpu_ray" /> -->
+      <!-- </xacro:if> -->
+      <!-- <xacro:unless value="${gpu}"> -->
+      <!--   <xacro:property name="ray_type" value="ray" /> -->
+      <!-- </xacro:unless> -->
       <gazebo reference="${frame_prefix}link">
         <sensor type="gpu_lidar" name="${frame_prefix}sensor">
           <topic>scan</topic>
+          <gz_frame_id>${frame_prefix}link</gz_frame_id>
           <pose>0.0 0.0 0.0 0.0 0.0 0.0</pose>
-          <visualize>false</visualize>
-		  <update_rate>12.5</update_rate>
-          <lidar>
+          <always_on>true</always_on>
+          <visualize>true</visualize>
+          <update_rate>12.5</update_rate>
+          <ray>
             <scan>
               <horizontal>
@@ -76,5 +78,5 @@
               <stddev>0.01</stddev>
             </noise>
-          </lidar>
+          </ray>
         </sensor>
       </gazebo>

File: robotnik_sensors/urdf/intel_d435.urdf.xacro (robot description, xacro)
@@ -8,26 +8,27 @@
   xmlns:xacro="http://wiki.ros.org/xacro">
   <!-- Includes -->
-  <xacro:macro name="sensor_intel_d435" params="prefix parent *origin prefix_topic:='front_rgbd_camera' use_nominal_extrinsics:=false">
+  <xacro:macro name="sensor_intel_d435"
+    params="prefix parent *origin prefix_topic:='front_rgbd_camera' use_nominal_extrinsics:=false">
     <xacro:property name="M_PI" value="3.1415926535897931" />
     <!-- The following values are approximate, and the camera node
      publishing TF values with actual calibrated camera extrinsic values -->
-    <xacro:property name="d435_cam_depth_to_infra1_offset" value="0.0"/>
-    <xacro:property name="d435_cam_depth_to_infra2_offset" value="-0.050"/>
-    <xacro:property name="d435_cam_depth_to_color_offset" value="0.015"/>
+    <xacro:property name="d435_cam_depth_to_infra1_offset" value="0.0" />
+    <xacro:property name="d435_cam_depth_to_infra2_offset" value="-0.050" />
+    <xacro:property name="d435_cam_depth_to_color_offset" value="0.015" />
     <!-- The following values model the aluminum peripherial case for the
     D435 camera, with the camera joint represented by the actual
     peripherial camera tripod mount -->
-    <xacro:property name="d435_cam_width" value="0.090"/>
-    <xacro:property name="d435_cam_height" value="0.025"/>
-    <xacro:property name="d435_cam_depth" value="0.02505"/>
-    <xacro:property name="d435_cam_mount_from_center_offset" value="0.0149"/>
+    <xacro:property name="d435_cam_width" value="0.090" />
+    <xacro:property name="d435_cam_height" value="0.025" />
+    <xacro:property name="d435_cam_depth" value="0.02505" />
+    <xacro:property name="d435_cam_mount_from_center_offset" value="0.0149" />
     <!-- The following offset is relative the the physical D435 camera peripherial
     camera tripod mount -->
-    <xacro:property name="d435_cam_depth_px" value="${d435_cam_mount_from_center_offset}"/>
-    <xacro:property name="d435_cam_depth_py" value="0.0175"/>
-    <xacro:property name="d435_cam_depth_pz" value="${d435_cam_height/2}"/>
+    <xacro:property name="d435_cam_depth_px" value="${d435_cam_mount_from_center_offset}" />
+    <xacro:property name="d435_cam_depth_py" value="0.0175" />
+    <xacro:property name="d435_cam_depth_pz" value="${d435_cam_height/2}" />
     <joint name="${prefix}_base_joint" type="fixed">
       <xacro:insert_block name="origin" />
-      <parent link="${parent}"/>
+      <parent link="${parent}" />
       <child link="${prefix}_base_link" />
     </joint>
@@ -37,19 +38,22 @@
       <parent link="${prefix}_base_link" />
       <child link="${prefix}_link" />
-      <origin xyz="0.01 0.02 0" rpy="0 0 0"/>
+      <origin xyz="0.01 0.02 0" rpy="0 0 0" />
       <child link="${prefix}_link" />
     </joint>
-    <link name="${prefix}_link"> <!-- camera link is aligned with the infrared sensor 1 that is "in the middle of the camera", not the one in the edge -->
+    <link name="${prefix}_link"> <!-- camera link is aligned with the infrared sensor 1 that is "in
+      the middle of the camera", not the one in the edge -->
       <visual>
-        <origin xyz="${d435_cam_mount_from_center_offset} ${-d435_cam_depth_py} 0" rpy="${M_PI/2} 0 ${M_PI/2}"/>
+        <origin xyz="${d435_cam_mount_from_center_offset} ${-d435_cam_depth_py} 0"
+          rpy="${M_PI/2} 0 ${M_PI/2}" />
         <geometry>
           <!-- <box size="${d435_cam_width} ${d435_cam_height} ${d435_cam_depth}"/> -->
-          <mesh filename="package://robotnik_sensors/meshes/depth/intel_realsense_d435/intel_d435_color.dae" />
+          <mesh
+            filename="package://robotnik_sensors/meshes/depth/intel_realsense_d435/intel_d435_color.dae" />
         </geometry>
       </visual>
       <collision>
-        <origin xyz="0 ${-d435_cam_depth_py} 0" rpy="0 0 0"/>
+        <origin xyz="0 ${-d435_cam_depth_py} 0" rpy="0 0 0" />
         <geometry>
-          <box size="${d435_cam_depth} ${d435_cam_width} ${d435_cam_height}"/>
+          <box size="${d435_cam_depth} ${d435_cam_width} ${d435_cam_height}" />
         </geometry>
       </collision>
@@ -60,13 +64,14 @@
       </inertial>
     </link>
-    <!-- Use the nominal extrinsics between camera frames if the calibrated extrinsics aren't being published. e.g. running the device in simulation  -->
+    <!-- Use the nominal extrinsics between camera frames if the calibrated extrinsics aren't being
+    published. e.g. running the device in simulation  -->
     <xacro:if value="${use_nominal_extrinsics}">
       <!-- camera depth joints and links -->
       <joint name="${prefix}_depth_joint" type="fixed">
-        <origin xyz="0 0 0" rpy="0 0 0"/>
-        <parent link="${prefix}_link"/>
+        <origin xyz="0 0 0" rpy="0 0 0" />
+        <parent link="${prefix}_link" />
         <child link="${prefix}_depth_frame" />
       </joint>
-      <link name="${prefix}_depth_frame"/>
+      <link name="${prefix}_depth_frame" />
       <joint name="${prefix}_depth_optical_joint" type="fixed">
         <origin xyz="0 0 0" rpy="${-M_PI/2} 0 ${-M_PI/2}" />
@@ -74,5 +79,5 @@
         <child link="${prefix}_depth_optical_frame" />
       </joint>
-      <link name="${prefix}_depth_optical_frame"/>
+      <link name="${prefix}_depth_optical_frame" />
       <!-- camera left IR joints and links -->
       <joint name="${prefix}_infra1_joint" type="fixed">
@@ -81,5 +86,5 @@
         <child link="${prefix}_infra1_frame" />
       </joint>
-      <link name="${prefix}_infra1_frame"/>
+      <link name="${prefix}_infra1_frame" />
       <joint name="${prefix}_infra1_optical_joint" type="fixed">
         <origin xyz="0 0 0" rpy="${-M_PI/2} 0 ${-M_PI/2}" />
@@ -87,5 +92,5 @@
         <child link="${prefix}_infra1_optical_frame" />
       </joint>
-      <link name="${prefix}_infra1_optical_frame"/>
+      <link name="${prefix}_infra1_optical_frame" />
       <!-- camera right IR joints and links -->
       <joint name="${prefix}_infra2_joint" type="fixed">
@@ -94,5 +99,5 @@
         <child link="${prefix}_infra2_frame" />
       </joint>
-      <link name="${prefix}_infra2_frame"/>
+      <link name="${prefix}_infra2_frame" />
       <joint name="${prefix}_infra2_optical_joint" type="fixed">
         <origin xyz="0 0 0" rpy="${-M_PI/2} 0 ${-M_PI/2}" />
@@ -100,5 +105,5 @@
         <child link="${prefix}_infra2_optical_frame" />
       </joint>
-      <link name="${prefix}_infra2_optical_frame"/>
+      <link name="${prefix}_infra2_optical_frame" />
       <!-- camera color joints and links -->
       <joint name="${prefix}_color_joint" type="fixed">
@@ -107,5 +112,5 @@
         <child link="${prefix}_color_frame" />
       </joint>
-      <link name="${prefix}_color_frame"/>
+      <link name="${prefix}_color_frame" />
       <joint name="${prefix}_color_optical_joint" type="fixed">
         <origin xyz="0 0 0" rpy="${-M_PI/2} 0 ${-M_PI/2}" />
@@ -113,121 +118,123 @@
         <child link="${prefix}_color_optical_frame" />
       </joint>
-      <link name="${prefix}_color_optical_frame"/>
+      <link name="${prefix}_color_optical_frame" />
     </xacro:if>
     <xacro:gazebo_d435 camera_name="${prefix}"
-                       reference_link="${prefix}_link"
-                       topics_ns="${prefix_topic}"
-                       depth_optical_frame="${prefix}_depth_optical_frame"
-                       color_optical_frame="${prefix}_color_optical_frame"
-                       infrared1_optical_frame="${prefix}_left_ir_optical_frame"
-                       infrared2_optical_frame="${prefix}_right_ir_optical_frame"/>
+      reference_link="${prefix}_link"
+      topics_ns="${prefix_topic}"
+      depth_optical_frame="${prefix}_depth_optical_frame"
+      color_optical_frame="${prefix}_color_optical_frame"
+      infrared1_optical_frame="${prefix}_left_ir_optical_frame"
+      infrared2_optical_frame="${prefix}_right_ir_optical_frame" />
   </xacro:macro>
-  <xacro:macro name="gazebo_d435" params="camera_name reference_link topics_ns depth_optical_frame color_optical_frame infrared1_optical_frame infrared2_optical_frame" >
-   <!-- Load parameters to model's main link-->
-   <xacro:property name="deg_to_rad" value="0.01745329251994329577" />
-   <gazebo reference="${reference_link}">
-     <self_collide>0</self_collide>
-     <enable_wind>0</enable_wind>
-     <kinematic>0</kinematic>
-     <gravity>1</gravity>
-     <!--<mu>1</mu>-->
-     <mu2>1</mu2>
-     <fdir1>0 0 0</fdir1>
-     <!--<slip1>0</slip1>
+  <xacro:macro name="gazebo_d435"
+    params="camera_name reference_link topics_ns depth_optical_frame color_optical_frame infrared1_optical_frame infrared2_optical_frame">
+    <!-- Load parameters to model's main link-->
+    <xacro:property name="deg_to_rad" value="0.01745329251994329577" />
+    <gazebo reference="${reference_link}">
+      <self_collide>0</self_collide>
+      <enable_wind>0</enable_wind>
+      <kinematic>0</kinematic>
+      <gravity>1</gravity>
+      <!--<mu>1</mu>-->
+      <mu2>1</mu2>
+      <fdir1>0 0 0</fdir1>
+      <!--<slip1>0</slip1>
      <slip2>0</slip2>-->
-     <kp>1e+13</kp>
-     <kd>1</kd>
-     <!--<max_vel>0.01</max_vel>
+      <kp>1e+13</kp>
+      <kd>1</kd>
+      <!--<max_vel>0.01</max_vel>
      <min_depth>0</min_depth>-->
-     <sensor name="${camera_name}color" type="camera">
-       <topic>camera/image_raw</topic>
-       <camera name="${camera_name}">
-         <horizontal_fov>${69.4*deg_to_rad}</horizontal_fov>
-         <image>
-           <width>1920</width>
-           <height>1080</height>
-           <format>RGB_INT8</format>
-         </image>
-         <clip>
-           <near>0.1</near>
-           <far>100</far>
-         </clip>
-         <noise>
-           <type>gaussian</type>
-           <mean>0.0</mean>
-           <stddev>0.007</stddev>
-         </noise>
-       </camera>
-       <always_on>1</always_on>
-       <update_rate>30</update_rate>
-       <visualize>false</visualize>
-     </sensor>
-     <sensor name="${camera_name}ired1" type="camera">
-       <camera name="${camera_name}">
-         <horizontal_fov>${85.2*deg_to_rad}</horizontal_fov>
-         <image>
-           <width>1280</width>
-           <height>720</height>
-           <format>L_INT8</format>
-         </image>
-         <clip>
-           <near>0.1</near>
-           <far>100</far>
-         </clip>
-         <noise>
-           <type>gaussian</type>
-           <mean>0.0</mean>
-           <stddev>0.05</stddev>
-         </noise>
-       </camera>
-       <always_on>1</always_on>
-       <update_rate>90</update_rate>
-       <visualize>false</visualize>
-     </sensor>
-     <sensor name="${camera_name}ired2" type="camera">
-       <camera name="${camera_name}">
-         <horizontal_fov>${85.2*deg_to_rad}</horizontal_fov>
-         <image>
-           <width>1280</width>
-           <height>720</height>
-           <format>L_INT8</format>
-         </image>
-         <clip>
-           <near>0.1</near>
-           <far>100</far>
-         </clip>
-         <noise>
-           <type>gaussian</type>
-           <mean>0.0</mean>
-           <stddev>0.05</stddev>
-         </noise>
-       </camera>
-       <always_on>1</always_on>
-       <update_rate>90</update_rate>
-       <visualize>false</visualize>
-     </sensor>
-     <sensor name="${camera_name}depth" type="depth">
-       <topic>camera/depth_image</topic>
-       <camera name="${camera_name}">
-         <horizontal_fov>${85.2*deg_to_rad}</horizontal_fov>
-         <image>
-           <width>1280</width>
-           <height>720</height>
-         </image>
-         <clip>
-           <near>0.1</near>
-           <far>100</far>
-         </clip>
-         <noise>
-           <type>gaussian</type>
-           <mean>0.0</mean>
-           <stddev>0.100</stddev>
-         </noise>
-       </camera>
-       <always_on>1</always_on>
-       <update_rate>90</update_rate>
-       <visualize>false</visualize>
-     </sensor>
-   </gazebo>
+      <sensor name="${camera_name}color" type="camera">
+        <topic>camera/image_raw</topic>
+        <camera name="${camera_name}">
+          <horizontal_fov>${69.4*deg_to_rad}</horizontal_fov>
+          <image>
+            <width>1920</width>
+            <height>1080</height>
+            <format>RGB_INT8</format>
+          </image>
+          <clip>
+            <near>0.1</near>
+            <far>100</far>
+          </clip>
+          <noise>
+            <type>gaussian</type>
+            <mean>0.0</mean>
+            <stddev>0.007</stddev>
+          </noise>
+        </camera>
+        <always_on>1</always_on>
+        <update_rate>30</update_rate>
+        <visualize>false</visualize>
+      </sensor>
+      <sensor name="${camera_name}ired1" type="camera">
+        <camera name="${camera_name}">
+          <horizontal_fov>${85.2*deg_to_rad}</horizontal_fov>
+          <image>
+            <width>1280</width>
+            <height>720</height>
+            <format>L_INT8</format>
+          </image>
+          <clip>
+            <near>0.1</near>
+            <far>100</far>
+          </clip>
+          <noise>
+            <type>gaussian</type>
+            <mean>0.0</mean>
+            <stddev>0.05</stddev>
+          </noise>
+        </camera>
+        <always_on>1</always_on>
+        <update_rate>90</update_rate>
+        <visualize>false</visualize>
+      </sensor>
+      <sensor name="${camera_name}ired2" type="camera">
+        <camera name="${camera_name}">
+          <horizontal_fov>${85.2*deg_to_rad}</horizontal_fov>
+          <image>
+            <width>1280</width>
+            <height>720</height>
+            <format>L_INT8</format>
+          </image>
+          <clip>
+            <near>0.1</near>
+            <far>100</far>
+          </clip>
+          <noise>
+            <type>gaussian</type>
+            <mean>0.0</mean>
+            <stddev>0.05</stddev>
+          </noise>
+        </camera>
+        <always_on>1</always_on>
+        <update_rate>90</update_rate>
+        <visualize>false</visualize>
+      </sensor>
+      <sensor name="${camera_name}depth" type="depth">
+        <topic>camera/depth_image</topic>
+        <gz_frame_id>${prefix}_link</gz_frame_id>
+        <camera name="${camera_name}">
+          <horizontal_fov>${85.2*deg_to_rad}</horizontal_fov>
+          <image>
+            <width>1280</width>
+            <height>720</height>
+          </image>
+          <clip>
+            <near>0.1</near>
+            <far>100</far>
+          </clip>
+          <noise>
+            <type>gaussian</type>
+            <mean>0.0</mean>
+            <stddev>0.100</stddev>
+          </noise>
+        </camera>
+        <always_on>1</always_on>
+        <update_rate>90</update_rate>
+        <visualize>false</visualize>
+      </sensor>
+    </gazebo>
   </xacro:macro>
 </robot>
